File: xDuinoRails-Thor-M.kicad_sch (KiCad schematic)
At the start: 1 part, among them U1101 MOUDLE-SEEEDUINO-XIAO

Commit message: Chg - Draft of Plux16 connector
Connections:
- no-connect marks 6 -> 1
Other:
- sheet loco-adapter-nem660-21mtc renamed loco-adapters-2func
- sheet loco-adapters-2func: file loco-adapter-nem660-21mtc.kicad_sch -> loco-adapters-2func.kicad_sch
- sheet loco-adapters-2func ports: added none; removed AMP_AUX[1..7], AUX89_ZBCLK, AUX910_ZBDATA, AUX[1..8], SPEAKER[0..1]
Changed lines of the file:
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@@
-	)
-	(no_connect
-		(at 261.62 102.87)
-	)
-	(no_connect
-		(at 226.06 115.57)
-	)
-	(no_connect
-		(at 261.62 107.95)
 	)
 	(no_connect
 		(at 129.54 115.57)
-	)
-	(no_connect
-		(at 261.62 100.33)
-	)
-	(no_connect
-		(at 226.06 111.76)
 	)
 	(bus_entry
@@
 			(color 255 253 198 1.0000)
 		)
-		(property "Sheetname" "loco-adapter-nem660-21mtc"
+		(property "Sheetname" "loco-adapters-2func"
 			(at 226.06 93.2684 0)
 			(effects
@@
 			)
 		)
-		(property "Sheetfile" "loco-adapter-nem660-21mtc.kicad_sch"
+		(property "Sheetfile" "loco-adapters-2func.kicad_sch"
 			(at 226.06 123.7746 0)
 			(effects
@@
 			)
 		)
-		(pin "AUX89_ZBCLK" input
-			(at 261.62 100.33 0)
-			(effects
-				(font
-					(size 1.27 1.27)
-				)
-				(justify right)
-			)
-		)
-		(pin "AUX910_ZBDATA" input
-			(at 261.62 102.87 0)
-			(effects
-				(font
-					(size 1.27 1.27)
-				)
-				(justify right)
-			)
-		)
 		(pin "+3V3" input
 			(at 242.57 93.98 90)
@@
 			)
 		)
-		(pin "SPEAKER[0..1]" input
-			(at 226.06 115.57 180)
-			(effects
-				(font
-					(size 1.27 1.27)
-				)
-				(justify left)
-			)
-		)
 		(pin "AMP_FUNC[0..1]" input
 			(at 226.06 107.95 180)
@@
 			)
 		)
-		(pin "AMP_AUX[1..7]" input
-			(at 226.06 111.76 180)
-			(effects
-				(font
-					(size 1.27 1.27)
-				)
-				(justify left)
-			)
-		)
 		(pin "AMP_MOTOR[0..1]" input
 			(at 226.06 104.14 180)
@@
 			(effects
 				(font
-					(size 1.27 1.27)
-				)
-				(justify right)
-			)
-		)
-		(pin "AUX[1..8]" input
-			(at 261.62 107.95 0)
-			(effects
-				(font
