File: xDuinoRails-Thor-M - Kopie.kicad_pcb (KiCad board)
At the start: 6 copper layers, 30 x 20.1 mm, 46 parts, among them J1101 Conn_02x08_Odd_Even, Q501 S8050, Q601 S8550, Q602 S8550, Q604 S8050, Q901 BSS138, Q902 BSS138, U1301 MOUDLE-SEEEDUINO-XIAO, U201 HT75xx-1-SOT89, U801 BDR6133

Commit message: Add - plux16 integration v0.9
Parts:
- moved R902 3.30 mm to (171.3, 94.0), turned to 180 degrees
- moved R901 3.30 mm to (168.0, 94.0), turned to 0 degrees
- moved TP404 2.54 mm to (171.3, 99.7)
- moved TP405 2.54 mm to (171.3, 102.2)
Routing:
- net /FUNC1: track 65.2 -> 32.8 mm, vias 3 -> 2
- net /DCC0: track 58.9 -> 32.8 mm, vias 6 -> 4
- net /AMP_FUNC1: track 19.3 -> 1.45 mm, vias 2 -> 1
- net /AMP_FUNC0: track 18.3 -> 1.49 mm, vias 3 -> 1
- net /AMP_MOTOR1: track 23.2 -> 8.40 mm, vias 2 -> 1
- net /MOTOR1: track 22.3 -> 13.2 mm
- net /AMP_MOTOR0: track 16.3 -> 7.94 mm, vias 2 -> 1
- net /+U: track 57.6 -> 50.3 mm
- net /EMF_MOTOR1: track 32.1 -> 26.7 mm
- net /MOTOR0: track 4.95 -> 7.27 mm
- net /+3V3: track 16.1 -> 14.6 mm
- net /FUNC0: track 30.9 -> 32.2 mm, vias 2 -> 3
- net /I_FUNC: track 27.8 -> 26.6 mm
- net /EMF_MOTOR0: track 25.9 -> 25.0 mm
- net /DCC1: track 52.5 -> 53.3 mm, vias 5 -> 4
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Other:
- board text added: "Fehlender PIN"
