File: loco-driver-motor.kicad_sch (KiCad schematic)
At the start: 20 parts, among them U801 BDR6133

Commit message: Fix - BOM errors
Parts:
- C802, C803: footprint Capacitor_SMD:C_0603_1608Metric_Pad1.08x0.95mm_HandSolder -> Capacitor_SMD:C_0805_2012Metric_Pad1.18x1.45mm_HandSolder
Changed lines of the file:
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@@
 			)
 		)
-		(property "Footprint" "Capacitor_SMD:C_0603_1608Metric_Pad1.08x0.95mm_HandSolder"
+		(property "Footprint" "Capacitor_SMD:C_0805_2012Metric_Pad1.18x1.45mm_HandSolder"
 			(at 81.5848 58.42 0)
 			(effects
@@
 			)
 		)
-		(property "Footprint" "Capacitor_SMD:C_0603_1608Metric_Pad1.08x0.95mm_HandSolder"
+		(property "Footprint" "Capacitor_SMD:C_0805_2012Metric_Pad1.18x1.45mm_HandSolder"
 			(at 47.9552 50.8 0)
 			(effects

Commit message: Fix - 100nF capacitor size
Parts:
- C801: OLI_ID 100nF_0603 -> 100nF_0805
Changed lines of the file:
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@@
 			)
 		)
-		(property "OLI_ID" "100nF_0603"
+		(property "OLI_ID" "100nF_0805"
 			(at 39.37 54.61 0)
 			(effects

Commit message: Fix - 3D model and some silkscreen
Parts:
- U801: footprint Package_SO:SOIC-8-1EP_3.9x4.9mm_P1.27mm_EP2.41x3.3mm_ThermalVias -> xDuinoRail:SOIC-8-1EP_3.9x4.9mm_P1.27mm_EP2.41x3.3mm_ThermalVias
Changed lines of the file:
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@@
 			)
 		)
-		(property "Footprint" "Package_SO:SOIC-8-1EP_3.9x4.9mm_P1.27mm_EP2.41x3.3mm_ThermalVias"
+		(property "Footprint" "xDuinoRail:SOIC-8-1EP_3.9x4.9mm_P1.27mm_EP2.41x3.3mm_ThermalVias"
 			(at 57.912 97.282 0)
 			(effects

Commit message: Fix - Component size for 100nF
Parts:
- C804: OLI_ID 100nF_0603 -> 100nF_0805
Changed lines of the file:
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@@
 			)
 		)
-		(property "OLI_ID" "100nF_0603"
+		(property "OLI_ID" "100nF_0805"
 			(at 90.17 54.61 0)
 			(effects
